File: PCB_Practice/PCB_AstMul.kicad_pcb (KiCad board)
At the start: 2 copper layers, 0 parts

Commit message: add EdgeCuts
Other:
- board outline added: 35 x 70 mm
Changed lines of the file:
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@@
 	)
 	(net 0 "")
+	(gr_rect
+		(start 130 70)
+		(end 165 140)
+		(stroke
+			(width 0.1)
+			(type default)
+		)
+		(fill no)
+		(layer "Edge.Cuts")
+	)
 	(embedded_fonts no)
 )
